File: IR_scrambler_circuit_kicad/IR_scrambler.sch (KiCad schematic (older format))
At the start: 11 parts, among them IC1 ATTINY85-P, P1 PROG HEADER, Q1 BC547, SW1 SW_Push

Commit message: Updated circuit schematics
Parts:
- SW1: value SW_Push -> ON/Cancel
Changed lines of the file:
@@
 P 4950 3450
 F 0 "SW1" H 5000 3550 50  0000 L CNN
-F 1 "SW_Push" H 4950 3390 50  0000 C CNN
+F 1 "ON/Cancel" H 4950 3390 50  0000 C CNN
 F 2 "" H 4950 3650 50  0000 C CNN
 F 3 "" H 4950 3650 50  0000 C CNN
